Commit message: feat: working robot model in gazebo

File: src/my_amr_sim/urdf/my_amr.urdf.xacro (robot description, xacro)
@@ -2,4 +2,6 @@
 <robot name="my_amr" xmlns:xacro="http://www.ros.org/wiki/xacro">
   <xacro:include filename="$(find my_amr_sim)/urdf/ros2_control.xacro"/>
+  <!-- Mesh scale: adjust if your STLs were exported in mm instead of meters -->
+  <xacro:property name="mesh_scale" value="0.001 0.001 0.001"/>
   <!-- ======================== Base ======================== -->
   <link name="base_footprint"/>
@@ -7,13 +9,17 @@
     <parent link="base_footprint"/>
     <child link="base_link"/>
-    <origin xyz="0 0 0.075"/>
+    <origin xyz="0 0 0.0826"/>
   </joint>
   <link name="base_link">
     <visual>
-      <geometry><box size="0.5 0.35 0.15"/></geometry>
+      <geometry>
+        <mesh filename="package://my_amr_sim/meshes/body.stl" scale="${mesh_scale}"/>
+      </geometry>
       <material name="blue"><color rgba="0.2 0.4 0.8 1"/></material>
     </visual>
     <collision>
-      <geometry><box size="0.5 0.35 0.15"/></geometry>
+      <geometry>
+        <mesh filename="package://my_amr_sim/meshes/body.stl" scale="${mesh_scale}"/>
+      </geometry>
     </collision>
     <inertial>
@@ -26,14 +32,18 @@
     <parent link="base_link"/>
     <child link="left_wheel"/>
-    <origin xyz="0 0.2 -0.025" rpy="-1.5708 0 0"/>
-    <axis xyz="0 0 1"/>
+    <origin xyz="0.230 0.0 0.0" rpy="-1.5708 0 0"/>
+    <axis xyz="1 0 0"/>
   </joint>
   <link name="left_wheel">
     <visual>
-      <geometry><cylinder radius="0.05" length="0.04"/></geometry>
-      <material name="dark"><color rgba="0.1 0.1 0.1 1"/></material>
-    </visual>
-    <collision>
-      <geometry><cylinder radius="0.05" length="0.04"/></geometry>
+      <geometry>
+        <mesh filename="package://my_amr_sim/meshes/wheel.stl" scale="${mesh_scale}"/>
+      </geometry>
+      <material name="dark"><color rgba="0.1 0.1 0.1 1"/></material>
+    </visual>
+    <collision>
+      <geometry>
+          <mesh filename="package://my_amr_sim/meshes/wheel.stl" scale="${mesh_scale}"/>
+        </geometry>
     </collision>
     <inertial>
@@ -45,14 +55,20 @@
     <parent link="base_link"/>
     <child link="right_wheel"/>
-    <origin xyz="0 -0.2 -0.025" rpy="1.5708 0 0"/>
-    <axis xyz="0 0 1"/>
+    <origin xyz="-0.230 0.0 0.0" rpy="1.5708 0 0"/>
+    <axis xyz="1 0 0"/>
   </joint>
   <link name="right_wheel">
     <visual>
-      <geometry><cylinder radius="0.05" length="0.04"/></geometry>
-      <material name="dark"><color rgba="0.1 0.1 0.1 1"/></material>
-    </visual>
-    <collision>
-      <geometry><cylinder radius="0.05" length="0.04"/></geometry>
+      <!-- rpy="0 3.14159 0" flips the mesh if the right side appears mirrored -->
+      <origin rpy="0 3.14159 0"/>
+      <geometry>
+        <mesh filename="package://my_amr_sim/meshes/wheel.stl" scale="${mesh_scale}"/>
+      </geometry>
+      <material name="dark"><color rgba="0.1 0.1 0.1 1"/></material>
+    </visual>
+    <collision>
+      <geometry>
+          <mesh filename="package://my_amr_sim/meshes/wheel.stl" scale="${mesh_scale}"/>
+        </geometry>
     </collision>
     <inertial>
@@ -62,54 +78,95 @@
   </link>
   <!-- ======================== Caster wheels ======================== -->
-  <joint name="front_caster_joint" type="fixed">
-    <parent link="base_link"/>
-    <child link="front_caster"/>
-    <origin xyz="0.2 0 -0.05"/>
-  </joint>
-  <link name="front_caster">
-    <visual>
-      <geometry><sphere radius="0.025"/></geometry>
-      <material name="dark"><color rgba="0.1 0.1 0.1 1"/></material>
-    </visual>
-    <collision>
-      <geometry><sphere radius="0.025"/></geometry>
-    </collision>
-    <inertial>
-      <mass value="0.1"/>
-      <inertia ixx="0.000025" ixy="0" ixz="0" iyy="0.000025" iyz="0" izz="0.000025"/>
-    </inertial>
-  </link>
-  <joint name="rear_caster_joint" type="fixed">
-    <parent link="base_link"/>
-    <child link="rear_caster"/>
-    <origin xyz="-0.2 0 -0.05"/>
-  </joint>
-  <link name="rear_caster">
-    <visual>
-      <geometry><sphere radius="0.025"/></geometry>
-      <material name="dark"><color rgba="0.1 0.1 0.1 1"/></material>
-    </visual>
-    <collision>
-      <geometry><sphere radius="0.025"/></geometry>
-    </collision>
-    <inertial>
-      <mass value="0.1"/>
-      <inertia ixx="0.000025" ixy="0" ixz="0" iyy="0.000025" iyz="0" izz="0.000025"/>
-    </inertial>
-  </link>
-  <!-- ======================== 2D Lidar ======================== -->
+  <joint name="front_left_caster_joint" type="fixed">
+    <parent link="base_link"/>
+    <child link="front_left_caster"/>
+    <origin xyz="0.210 0.335 -0.031"/>
+  </joint>
+  <link name="front_left_caster">
+    <visual>
+      <geometry><sphere radius="0.05"/></geometry>
+      <material name="dark"><color rgba="0.1 0.1 0.1 1"/></material>
+    </visual>
+    <collision>
+      <geometry><sphere radius="0.05"/></geometry>
+    </collision>
+    <inertial>
+      <mass value="0.1"/>
+      <inertia ixx="0.000025" ixy="0" ixz="0" iyy="0.000025" iyz="0" izz="0.000025"/>
+    </inertial>
+  </link>
+  <joint name="rear_left_caster_joint" type="fixed">
+    <parent link="base_link"/>
+    <child link="rear_left_caster"/>
+    <origin xyz="-0.210 0.335 -0.031"/>
+  </joint>
+  <link name="rear_left_caster">
+    <visual>
+      <geometry><sphere radius="0.05"/></geometry>
+      <material name="dark"><color rgba="0.1 0.1 0.1 1"/></material>
+    </visual>
+    <collision>
+      <geometry><sphere radius="0.05"/></geometry>
+    </collision>
+    <inertial>
+      <mass value="0.1"/>
+      <inertia ixx="0.000025" ixy="0" ixz="0" iyy="0.000025" iyz="0" izz="0.000025"/>
+    </inertial>
+  </link>
+  <joint name="front_right_caster_joint" type="fixed">
+    <parent link="base_link"/>
+    <child link="front_right_caster"/>
+    <origin xyz="0.210 -0.335 -0.031"/>
+  </joint>
+  <link name="front_right_caster">
+    <visual>
+      <geometry><sphere radius="0.05"/></geometry>
+      <material name="dark"><color rgba="0.1 0.1 0.1 1"/></material>
+    </visual>
+    <collision>
+      <geometry><sphere radius="0.05"/></geometry>
+    </collision>
+    <inertial>
+      <mass value="0.1"/>
+      <inertia ixx="0.000025" ixy="0" ixz="0" iyy="0.000025" iyz="0" izz="0.000025"/>
+    </inertial>
+  </link>
+  <joint name="rear_right_caster_joint" type="fixed">
+    <parent link="base_link"/>
+    <child link="rear_right_caster"/>
+    <origin xyz="-0.210 -0.335 -0.031"/>
+  </joint>
+  <link name="rear_right_caster">
+    <visual>
+      <geometry><sphere radius="0.05"/></geometry>
+      <material name="dark"><color rgba="0.1 0.1 0.1 1"/></material>
+    </visual>
+    <collision>
+      <geometry><sphere radius="0.05"/></geometry>
+    </collision>
+    <inertial>
+      <mass value="0.1"/>
+      <inertia ixx="0.000025" ixy="0" ixz="0" iyy="0.000025" iyz="0" izz="0.000025"/>
+    </inertial>
+  </link>
+  <!-- ======================== RPLidar S2 ======================== -->
   <joint name="lidar_joint" type="fixed">
     <parent link="base_link"/>
     <child link="lidar_link"/>
-    <origin xyz="0.15 0 0.1"/>
+    <!-- lidar_link = scan plane: mount height (0.08) + sensor height (0.039) -->
+    <origin xyz="0.0 -0.400 0.110"/>
   </joint>
   <link name="lidar_link">
     <visual>
-      <geometry><cylinder radius="0.03" length="0.05"/></geometry>
-      <material name="black"><color rgba="0 0 0 1"/></material>
-    </visual>
-    <inertial>
-      <mass value="0.1"/>
-      <inertia ixx="0.000025" ixy="0" ixz="0" iyy="0.000025" iyz="0" izz="0.000025"/>
+      <!-- mesh Z starts at 0 (sensor base); shift down so it renders below the scan frame -->
+      <origin xyz="0 0 -0.030"/>
+      <geometry>
+        <mesh filename="package://my_amr_sim/meshes/rplidar_s2.stl" scale="${mesh_scale}"/>
+      </geometry>
+      <material name="dark"><color rgba="0.1 0.1 0.1 1"/></material>
+    </visual>
+    <inertial>
+      <mass value="0.185"/>
+      <inertia ixx="0.0001" ixy="0" ixz="0" iyy="0.0001" iyz="0" izz="0.0001"/>
     </inertial>
   </link>
@@ -117,10 +174,10 @@
     <sensor name="lidar" type="gpu_lidar">
       <topic>scan</topic>
-      <update_rate>10</update_rate>
+      <update_rate>15</update_rate>
       <gz_frame_id>lidar_link</gz_frame_id>
       <lidar>
         <scan>
           <horizontal>
-            <samples>360</samples>
+            <samples>720</samples>
             <min_angle>-3.14159</min_angle>
             <max_angle>3.14159</max_angle>
@@ -128,20 +185,72 @@
         </scan>
         <range>
-          <min>0.1</min>
-          <max>12.0</max>
+          <min>0.05</min>
+          <max>30.0</max>
+          <resolution>0.01</resolution>
         </range>
       </lidar>
       <always_on>true</always_on>
-      <visualize>true</visualize>
+      <visualize>false</visualize>
     </sensor>
   </gazebo>
-  <!-- Caster wheel friction -->
-  <gazebo reference="front_caster">
-    <mu1>0.0</mu1>
-    <mu2>0.0</mu2>
-  </gazebo>
-  <gazebo reference="rear_caster">
-    <mu1>0.0</mu1>
-    <mu2>0.0</mu2>
+  <!-- ======================== Ellipse Micro AHRS (IMU) ======================== -->
+  <joint name="imu_joint" type="fixed">
+    <parent link="base_link"/>
+    <child link="imu_link"/>
+    <origin xyz="0 0 0.0"/>
+  </joint>
+  <link name="imu_link">
+    <visual>
+      <geometry>
+        <mesh filename="package://my_amr_sim/meshes/ellipse_micro_ahrs.stl" scale="${mesh_scale}"/>
+      </geometry>
+      <material name="dark"><color rgba="0.1 0.1 0.1 1"/></material>
+    </visual>
+    <inertial>
+      <mass value="0.017"/>
+      <inertia ixx="0.000001" ixy="0" ixz="0" iyy="0.000001" iyz="0" izz="0.000001"/>
+    </inertial>
+  </link>
+  <gazebo reference="imu_link">
+    <sensor name="imu" type="imu">
+      <topic>imu</topic>
+      <update_rate>100</update_rate>
+      <gz_frame_id>imu_link</gz_frame_id>
+      <imu>
+        <angular_velocity>
+          <x><noise type="gaussian"><mean>0</mean><stddev>0.009</stddev></noise></x>
+          <y><noise type="gaussian"><mean>0</mean><stddev>0.009</stddev></noise></y>
+          <z><noise type="gaussian"><mean>0</mean><stddev>0.009</stddev></noise></z>
+        </angular_velocity>
+        <linear_acceleration>
+          <x><noise type="gaussian"><mean>0</mean><stddev>0.021</stddev></noise></x>
+          <y><noise type="gaussian"><mean>0</mean><stddev>0.021</stddev></noise></y>
+          <z><noise type="gaussian"><mean>0</mean><stddev>0.021</stddev></noise></z>
+        </linear_acceleration>
+      </imu>
+      <always_on>true</always_on>
+      <visualize>false</visualize>
+    </sensor>
+  </gazebo>
+  <!-- ======================== Gazebo extras ======================== -->
+  <gazebo reference="left_wheel">
+    <mu1>1.0</mu1>
+    <mu2>1.0</mu2>
+  </gazebo>
+  <gazebo reference="right_wheel">
+    <mu1>1.0</mu1>
+    <mu2>1.0</mu2>
+  </gazebo>
+  <gazebo reference="front_left_caster">
+    <mu1>0.0</mu1><mu2>0.0</mu2>
+  </gazebo>
+  <gazebo reference="rear_left_caster">
+    <mu1>0.0</mu1><mu2>0.0</mu2>
+  </gazebo>
+  <gazebo reference="front_right_caster">
+    <mu1>0.0</mu1><mu2>0.0</mu2>
+  </gazebo>
+  <gazebo reference="rear_right_caster">
+    <mu1>0.0</mu1><mu2>0.0</mu2>
   </gazebo>
   <!-- ======================== ros2_control ======================== -->
