Commit message: feat: finalized the simulation skeleton

File: src/my_amr_sim/urdf/my_amr.urdf.xacro (robot description, xacro)
@@ -13,12 +13,14 @@
   <link name="base_link">
     <visual>
-      <geometry>
-        <mesh filename="package://my_amr_sim/meshes/body.stl" scale="${mesh_scale}"/>
+      <origin rpy="0 0 0.0"/>
+      <geometry>
+        <mesh filename="package://my_amr_sim/meshes/body_ccw_90.stl" scale="${mesh_scale}"/>
       </geometry>
       <material name="blue"><color rgba="0.2 0.4 0.8 1"/></material>
     </visual>
     <collision>
-      <geometry>
-        <mesh filename="package://my_amr_sim/meshes/body.stl" scale="${mesh_scale}"/>
+      <origin rpy="0 0 0.0"/>
+      <geometry>
+        <mesh filename="package://my_amr_sim/meshes/body_ccw_90.stl" scale="${mesh_scale}"/>
       </geometry>
     </collision>
@@ -32,17 +34,19 @@
     <parent link="base_link"/>
     <child link="left_wheel"/>
-    <origin xyz="0.230 0.0 0.0" rpy="-1.5708 0 0"/>
-    <axis xyz="1 0 0"/>
+    <origin xyz="0.0 0.230 0.0" rpy="1.5708 0 0"/>
+    <axis xyz="0 0 1"/>
   </joint>
   <link name="left_wheel">
     <visual>
-      <geometry>
-        <mesh filename="package://my_amr_sim/meshes/wheel.stl" scale="${mesh_scale}"/>
-      </geometry>
-      <material name="dark"><color rgba="0.1 0.1 0.1 1"/></material>
-    </visual>
-    <collision>
-      <geometry>
-          <mesh filename="package://my_amr_sim/meshes/wheel.stl" scale="${mesh_scale}"/>
+      <origin rpy="0 0 0"/>
+      <geometry>
+        <mesh filename="package://my_amr_sim/meshes/wheel_y_ccw_90.stl" scale="${mesh_scale}"/>
+      </geometry>
+      <material name="dark"><color rgba="0.1 0.1 0.1 1"/></material>
+    </visual>
+    <collision>
+      <origin rpy="0 0 0"/>
+      <geometry>
+          <mesh filename="package://my_amr_sim/meshes/wheel_y_ccw_90.stl" scale="${mesh_scale}"/>
         </geometry>
     </collision>
@@ -55,19 +59,19 @@
     <parent link="base_link"/>
     <child link="right_wheel"/>
-    <origin xyz="-0.230 0.0 0.0" rpy="1.5708 0 0"/>
-    <axis xyz="1 0 0"/>
+    <origin xyz="0.0 -0.230 0.0" rpy="-1.5708 0 0"/>
+    <axis xyz="0 0 1"/>
   </joint>
   <link name="right_wheel">
     <visual>
       <!-- rpy="0 3.14159 0" flips the mesh if the right side appears mirrored -->
-      <origin rpy="0 3.14159 0"/>
-      <geometry>
-        <mesh filename="package://my_amr_sim/meshes/wheel.stl" scale="${mesh_scale}"/>
-      </geometry>
-      <material name="dark"><color rgba="0.1 0.1 0.1 1"/></material>
-    </visual>
-    <collision>
-      <geometry>
-          <mesh filename="package://my_amr_sim/meshes/wheel.stl" scale="${mesh_scale}"/>
+      <origin rpy="0 0 0"/>
+      <geometry>
+        <mesh filename="package://my_amr_sim/meshes/wheel_y_ccw_90.stl" scale="${mesh_scale}"/>
+      </geometry>
+      <material name="dark"><color rgba="0.1 0.1 0.1 1"/></material>
+    </visual>
+    <collision>
+      <geometry>
+          <mesh filename="package://my_amr_sim/meshes/wheel_y_ccw_90.stl" scale="${mesh_scale}"/>
         </geometry>
     </collision>
@@ -81,5 +85,5 @@
     <parent link="base_link"/>
     <child link="front_left_caster"/>
-    <origin xyz="0.210 0.335 -0.031"/>
+    <origin xyz=" 0.335 0.210 -0.031"/>
   </joint>
   <link name="front_left_caster">
@@ -99,5 +103,5 @@
     <parent link="base_link"/>
     <child link="rear_left_caster"/>
-    <origin xyz="-0.210 0.335 -0.031"/>
+    <origin xyz="0.335 -0.210 -0.031"/>
   </joint>
   <link name="rear_left_caster">
@@ -117,5 +121,5 @@
     <parent link="base_link"/>
     <child link="front_right_caster"/>
-    <origin xyz="0.210 -0.335 -0.031"/>
+    <origin xyz="-0.335 0.210 -0.031"/>
   </joint>
   <link name="front_right_caster">
@@ -135,5 +139,5 @@
     <parent link="base_link"/>
     <child link="rear_right_caster"/>
-    <origin xyz="-0.210 -0.335 -0.031"/>
+    <origin xyz="-0.335 -0.210 -0.031"/>
   </joint>
   <link name="rear_right_caster">
@@ -154,6 +158,6 @@
     <parent link="base_link"/>
     <child link="lidar_link"/>
-    <!-- lidar_link = scan plane: mount height (0.08) + sensor height (0.039) -->
-    <origin xyz="0.0 -0.400 0.110"/>
+    <!-- lidar body mount: mount height (0.08) + sensor height (0.039) -->
+    <origin xyz="0.400 0 0.110"/>
   </joint>
   <link name="lidar_link">
@@ -162,5 +166,5 @@
       <origin xyz="0 0 -0.030"/>
       <geometry>
-        <mesh filename="package://my_amr_sim/meshes/rplidar_s2.stl" scale="${mesh_scale}"/>
+        <mesh filename="package://my_amr_sim/meshes/rplidar_s2_frame_aligned.stl" scale="${mesh_scale}"/>
       </geometry>
       <material name="dark"><color rgba="0.1 0.1 0.1 1"/></material>
@@ -203,5 +207,5 @@
     <visual>
       <geometry>
-        <mesh filename="package://my_amr_sim/meshes/ellipse_micro_ahrs.stl" scale="${mesh_scale}"/>
+        <mesh filename="package://my_amr_sim/meshes/ellipse_micro_ahrs_ccw_90.stl" scale="${mesh_scale}"/>
       </geometry>
       <material name="dark"><color rgba="0.1 0.1 0.1 1"/></material>
